File: LNA.sch (EAGLE design)
At the start: 54 parts, among them IC1 LM4562, IC4 DCDC, Q1 nmos, Q2 JFET-DUAL, Q3 NPN, Q4 PNP, SW1 SW

Commit message: 微修正
Parts:
- added C15: 10p, my_rcl:C-1608
- added DR1, DR2, DR3, DR4: HOLE-3.2, my_connector:HOLE-3.2
- added FB5: FB, my_rcl:FB-1608FB
- added Q5: 2SK2145, my_ic:JFET-DUAL
- added R14, R15: 3.6k, my_rcl:R-1608
- added R16: DNP, my_rcl:R-1608
- C1: value 10u -> 3.3u
- C2: value 10u -> 22u
- D1, D2: value D -> BIAS
- D4, D5: value (none) -> CLAMP
- Q1: value nmos -> BS138
- Q2: value JFET-DUAL -> 2SK2145
- R1: value 1k -> 360
Connections:
- new net N$8: FB5.2, Q2.G2, Q5.G1
- net +5V: now also R14.2, R15.2
- net -5V: now also R16.1
- net GND: now also C15.1
- net N$2: now also R16.2
- net N$21: now also Q5.S
- net N$24: now also Q2.D2, Q5.D1, R14.1; no longer Q2.D1
- net N$4: now also FB5.1; no longer Q2.G1, R3.2
- net N$5: now also R3.2
- net N$7: now also C15.2, Q2.D1, Q5.D2, R15.1; no longer Q2.D2
- net N$9: now also Q2.G1, Q5.G2; no longer Q2.G2
Other:
- moved on the sheet: C1, D4, D5, IC1G$3, R2, R3
